File: esquemas/Esquema_general.sch (EAGLE design)
At the start: 19 parts

Commit message: Actualización
Se han terminado de crear los componentes situados actualmente en el maletero del vehículo.
Falta terminar de crear los de la parte frontal, el monitor y el cableado.
Parts:
- added U$16: PC, ecar:PC
- added U$21: POWERBOX, ecar:POWERBOX
- added U$22: FUENTE_12V, ecar:FUENTE_12V
- added U$23: FUENTE_24V, ecar:FUENTE_24V
- added U$24: GPS, ecar:GPS
- added U$25: PHIDGETS_ENCODER, ecar:PHIDGETS_ENCODER
- added U$26, U$27: ENCODER_YUMO, ecar:ENCODER_YUMO
Other:
- moved on the sheet: U$7
Changed lines of the file:
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@@
 <setting verticaltext="up"/>
 </settings>
-<grid distance="0.1" unitdist="inch" unit="mm" style="lines" multiple="1" display="no" altdistance="0.01" altunitdist="inch" altunit="mm"/>
+<grid distance="0.1" unitdist="inch" unit="inch" style="lines" multiple="1" display="no" altdistance="0.01" altunitdist="inch" altunit="inch"/>
 <layers>
 <layer number="1" name="Top" color="4" fill="1" visible="no" active="no"/>
@@
 <part name="U$6" library="ecar" deviceset="VOLTIMETRO" device=""/>
 <part name="U$7" library="ecar" deviceset="CURTIS" device=""/>
+<part name="U$17" library="ecar" deviceset="AMPERIMETRO" device=""/>
+<part name="U$18" library="ecar" deviceset="AMPERIMETRO" device=""/>
+<part name="U$19" library="ecar" deviceset="AMPERIMETRO" device=""/>
+<part name="U$20" library="ecar" deviceset="AMPERIMETRO" device=""/>
 <part name="U$8" library="ecar" deviceset="BATERIA" device=""/>
 <part name="U$9" library="ecar" deviceset="BATERIA" device=""/>
@@
 <part name="U$14" library="ecar" deviceset="BATERIA" device=""/>
 <part name="U$15" library="ecar" deviceset="BATERIA" device=""/>
-<part name="U$17" library="ecar" deviceset="AMPERIMETRO" device=""/>
-<part name="U$18" library="ecar" deviceset="AMPERIMETRO" device=""/>
-<part name="U$19" library="ecar" deviceset="AMPERIMETRO" device=""/>
-<part name="U$20" library="ecar" deviceset="AMPERIMETRO" device=""/>
+<part name="U$21" library="ecar" deviceset="POWERBOX" device=""/>
+<part name="U$22" library="ecar" deviceset="FUENTE_12V" device=""/>
+<part name="U$23" library="ecar" deviceset="FUENTE_24V" device=""/>
+<part name="U$24" library="ecar" deviceset="GPS" device=""/>
+<part name="U$25" library="ecar" deviceset="PHIDGETS_ENCODER" device=""/>
+<part name="U$16" library="ecar" deviceset="PC" device=""/>
+<part name="U$26" library="ecar" deviceset="ENCODER_YUMO" device=""/>
+<part name="U$27" library="ecar" deviceset="ENCODER_YUMO" device=""/>
 </parts>
 <sheets>
@@
 </plain>
 <instances>
-<instance part="U$1" gate="G$1" x="662.94" y="276.86" rot="R90"/>
-<instance part="U$2" gate="G$1" x="165.1" y="187.96"/>
-<instance part="U$3" gate="G$1" x="629.92" y="68.58" rot="R180"/>
-<instance part="U$4" gate="G$1" x="215.9" y="215.9"/>
-<instance part="U$5" gate="G$1" x="231.14" y="215.9"/>
-<instance part="U$6" gate="G$1" x="246.38" y="215.9"/>
-<instance part="U$7" gate="G$1" x="525.78" y="88.9" rot="R180"/>
-<instance part="U$8" gate="G$1" x="213.36" y="175.26" rot="R90"/>
-<instance part="U$9" gate="G$1" x="213.36" y="154.94" rot="R90"/>
-<instance part="U$10" gate="G$1" x="213.36" y="137.16" rot="R90"/>
-<instance part="U$11" gate="G$1" x="213.36" y="119.38" rot="R90"/>
-<instance part="U$12" gate="G$1" x="213.36" y="99.06" rot="R90"/>
-<instance part="U$13" gate="G$1" x="213.36" y="78.74" rot="R90"/>
-<instance part="U$14" gate="G$1" x="213.36" y="58.42" rot="R90"/>
-<instance part="U$15" gate="G$1" x="213.36" y="40.64" rot="R90"/>
-<instance part="U$17" gate="G$1" x="563.88" y="-22.86" rot="R90"/>
-<instance part="U$18" gate="G$1" x="561.34" y="2.54" rot="R90"/>
-<instance part="U$19" gate="G$1" x="596.9" y="0" rot="R90"/>
-<instance part="U$20" gate="G$1" x="599.44" y="-22.86" rot="R90"/>
+<instance part="U$1" gate="G$1" x="1300.48" y="474.98" rot="R90"/>
+<instance part="U$2" gate="G$1" x="152.4" y="535.94"/>
+<instance part="U$3" gate="G$1" x="1320.8" y="165.1" rot="R180"/>
+<instance part="U$4" gate="G$1" x="187.96" y="546.1"/>
+<instance part="U$5" gate="G$1" x="205.74" y="546.1"/>
+<instance part="U$6" gate="G$1" x="223.52" y="546.1"/>
+<instance part="U$7" gate="G$1" x="1247.14" y="342.9" rot="R180"/>
+<instance part="U$17" gate="G$1" x="1325.88" y="-5.08" rot="R90"/>
+<instance part="U$18" gate="G$1" x="1280.16" y="45.72" rot="R90"/>
+<instance part="U$19" gate="G$1" x="1330.96" y="45.72" rot="R90"/>
+<instance part="U$20" gate="G$1" x="1277.62" y="7.62" rot="R90"/>
+<instance part="U$8" gate="G$1" x="789.94" y="391.16" rot="R90"/>
+<instance part="U$9" gate="G$1" x="792.48" y="251.46" rot="R90"/>
+<instance part="U$10" gate="G$1" x="1013.46" y="251.46" rot="R90"/>
+<instance part="U$11" gate="G$1" x="1016" y="109.22" rot="R90"/>
+<instance part="U$12" gate="G$1" x="601.98" y="248.92" rot="R90"/>
+<instance part="U$13" gate="G$1" x="1010.92" y="391.16" rot="R90"/>
+<instance part="U$14" gate="G$1" x="599.44" y="391.16" rot="R90"/>
+<instance part="U$15" gate="G$1" x="1010.92" y="525.78" rot="R90"/>
+<instance part="U$21" gate="G$1" x="165.1" y="508" rot="R270"/>
+<instance part="U$22" gate="G$1" x="0" y="497.84" rot="R270"/>
+<instance part="U$23" gate="G$1" x="335.28" y="574.04" rot="R180"/>
+<instance part="U$24" gate="G$1" x="73.66" y="307.34" rot="R270"/>
+<instance part="U$25" gate="G$1" x="251.46" y="180.34" rot="R90"/>
+<instance part="U$16" gate="G$1" x="7.62" y="5.08"/>
+<instance part="U$26" gate="G$1" x="198.12" y="632.46"/>
+<instance part="U$27" gate="G$1" x="238.76" y="-40.64" rot="R180"/>
 </instances>
 <busses>
@@
 </schematic>
 </drawing>
+<compatibility>
+<note version="6.3" minversion="6.2.2" severity="warning">
+Since Version 6.2.2 text objects can contain more than one line,
+which will not be processed correctly with this version.
+</note>
+</compatibility>
 </eagle>

Commit message: Suma de componentes
Parts:
- added U$28: MONITOR, ecar:MONITOR
- added U$29: SICK, ecar:SICK
Changed lines of the file:
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@@
 <part name="U$26" library="ecar" deviceset="ENCODER_YUMO" device=""/>
 <part name="U$27" library="ecar" deviceset="ENCODER_YUMO" device=""/>
+<part name="U$28" library="ecar" deviceset="MONITOR" device=""/>
+<part name="U$29" library="ecar" deviceset="SICK" device=""/>
 </parts>
 <sheets>
@@
 <instance part="U$26" gate="G$1" x="198.12" y="632.46"/>
 <instance part="U$27" gate="G$1" x="238.76" y="-40.64" rot="R180"/>
+<instance part="U$28" gate="G$1" x="1087.12" y="284.48" rot="R270"/>
+<instance part="U$29" gate="G$1" x="1363.98" y="327.66" rot="R270"/>
 </instances>
 <busses>

Commit message: Creación de componentes
Se terminan de crear los componentes existentes actualmente en el vehículo
Parts:
- added U$30: MOTOR_SENSORES, ecar:MOTOR_SENSORES
- added U$31: RASPBERRY_PI_3B, ecar:RASPBERRY_PI_3B
- added U$32: ARDUINO_PRO, ecar:ARDUINO_PRO
- added U$33: CONVERSOR_ARDUINO, ecar:CONVERSOR_ARDUINO
- added U$34: POLOLU_HIGH-POWER_MOTOR_DRIVER, ecar:POLOLU_HIGH-POWER_MOTOR_DRIVER
Other:
- moved on the sheet: U$7
Changed lines of the file:
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@@
 </classes>
 <parts>
-<part name="U$1" library="ecar" deviceset="MOTOR_DIRECCION" device=""/>
 <part name="U$2" library="ecar" deviceset="DAQ_NI" device=""/>
 <part name="U$3" library="ecar" deviceset="SENSOR_VELOCIDAD" device=""/>
@@
 <part name="U$28" library="ecar" deviceset="MONITOR" device=""/>
 <part name="U$29" library="ecar" deviceset="SICK" device=""/>
+<part name="U$30" library="ecar" deviceset="MOTOR_SENSORES" device=""/>
+<part name="U$31" library="ecar" deviceset="RASPBERRY_PI_3B" device=""/>
+<part name="U$1" library="ecar" deviceset="MOTOR_DIRECCION" device=""/>
+<part name="U$32" library="ecar" deviceset="ARDUINO_PRO" device=""/>
+<part name="U$33" library="ecar" deviceset="CONVERSOR_ARDUINO" device=""/>
+<part name="U$34" library="ecar" deviceset="POLOLU_HIGH-POWER_MOTOR_DRIVER" device=""/>
 </parts>
 <sheets>
@@
 </plain>
 <instances>
-<instance part="U$1" gate="G$1" x="1300.48" y="474.98" rot="R90"/>
 <instance part="U$2" gate="G$1" x="152.4" y="535.94"/>
-<instance part="U$3" gate="G$1" x="1320.8" y="165.1" rot="R180"/>
+<instance part="U$3" gate="G$1" x="1338.58" y="-25.4" rot="R180"/>
 <instance part="U$4" gate="G$1" x="187.96" y="546.1"/>
 <instance part="U$5" gate="G$1" x="205.74" y="546.1"/>
 <instance part="U$6" gate="G$1" x="223.52" y="546.1"/>
-<instance part="U$7" gate="G$1" x="1247.14" y="342.9" rot="R180"/>
-<instance part="U$17" gate="G$1" x="1325.88" y="-5.08" rot="R90"/>
-<instance part="U$18" gate="G$1" x="1280.16" y="45.72" rot="R90"/>
-<instance part="U$19" gate="G$1" x="1330.96" y="45.72" rot="R90"/>
-<instance part="U$20" gate="G$1" x="1277.62" y="7.62" rot="R90"/>
+<instance part="U$7" gate="G$1" x="1186.18" y="218.44" rot="R180"/>
+<instance part="U$17" gate="G$1" x="1176.02" y="-45.72" rot="R90"/>
+<instance part="U$18" gate="G$1" x="1176.02" y="-20.32" rot="R90"/>
+<instance part="U$19" gate="G$1" x="1176.02" y="5.08" rot="R90"/>
+<instance part="U$20" gate="G$1" x="764.54" y="53.34" rot="R90"/>
 <instance part="U$8" gate="G$1" x="789.94" y="391.16" rot="R90"/>
 <instance part="U$9" gate="G$1" x="792.48" y="251.46" rot="R90"/>
@@
 <instance part="U$27" gate="G$1" x="238.76" y="-40.64" rot="R180"/>
 <instance part="U$28" gate="G$1" x="1087.12" y="284.48" rot="R270"/>
-<instance part="U$29" gate="G$1" x="1363.98" y="327.66" rot="R270"/>
+<instance part="U$29" gate="G$1" x="1584.96" y="327.66" rot="R270"/>
+<instance part="U$30" gate="G$1" x="1435.1" y="-22.86" rot="R90"/>
+<instance part="U$31" gate="G$1" x="1231.9" y="388.62"/>
+<instance part="U$1" gate="G$1" x="1422.4" y="541.02" rot="R90"/>
+<instance part="U$32" gate="G$1" x="1270" y="482.6"/>
+<instance part="U$33" gate="G$1" x="1252.22" y="502.92" rot="R180"/>
+<instance part="U$34" gate="G$1" x="1097.28" y="497.84"/>
 </instances>
 <busses>

Commit message: Diagrama baterías
Finalizada la representación del cableado de la zona de baterías. Cables de cada batería y de la manguera de cables de los dos amperímetros instalados.
Parts:
- added U$35: AMPERIMETRO, ecar:AMPERIMETRO
Connections:
- new net AMARILLO_OUTPUT_HONEYWELL: U$35.VOUT
- new net BAT_1: U$35.IN, U$9.-VCC
- new net BAT_1+: U$11.+VCC, U$20.OUT
- new net BAT_2+: U$10.+VCC, U$11.-VCC
- new net BAT_3+: U$10.-VCC, U$13.+VCC
- new net BAT_4+: U$13.-VCC, U$15.+VCC
- new net BAT_6+: U$12.-VCC, U$9.+VCC
- new net BAT_7+: U$14.+VCC, U$8.-VCC
- new net BAT_8+: U$12.+VCC, U$14.-VCC
- new net BLANCO_VCC_LEM: U$20.VCC
- new net MARRON_VCC_HONEYWELL: U$35.VCC
- new net N$1: U$15.-VCC, U$8.+VCC
- new net N$2: U$20.IN, U$35.OUT
- new net NEGRO_-VCC_HONEYWELL: U$35.GND
- new net ROJO_VOUT_LEM: U$20.VOUT
- new net VERDE_GND_LEM: U$20.GND
Other:
- note added: "ZONA INFERIOR ECARM"

Commit message: Conexión de componentes del maletero.
Aún no está terminado.
Parts:
- removed U$17: AMPERIMETRO, ecar:AMPERIMETRO
Connections:
- new net 5V_GND: U$21.GND(5V)
- new net 5V_VCC: U$21.+5V
- new net ENC_L_5V: U$25.E0_5V, U$26.5-12V
- new net ENC_L_COMMON: U$26.COMMON
- new net ENC_L_GND: U$25.E0_GND, U$26.GND
- new net ENC_L_OUT_A: U$25.E0_A, U$26.OUT_A
- new net ENC_L_OUT_B: U$25.E0_B, U$26.OUT_B
- new net ENC_L_OUT_Z: U$25.E0_INDEX, U$26.OUT_Z
- new net ENC_R_5V: U$25.E1_5V, U$27.5-12V
- new net ENC_R_COMMON: U$27.COMMON
- new net ENC_R_GND: U$25.E1_GND, U$27.GND
- new net ENC_R_OUT_A: U$25.E1_A, U$27.OUT_A
- new net ENC_R_OUT_B: U$25.E1_B, U$27.OUT_B
- new net ENC_R_OUT_Z: U$25.E1_INDEX, U$27.OUT_Z
- new net ORDENADOR_GND: U$16.GND, U$21.OUT-3
- new net ORDENADOR_VCC: U$16.VCC, U$21.OUT+3
- new net USB_PHIDGET_ENCODER_PC: U$16.USB1, U$25.USB
- net BAT_1: now also U$21.IN_GND
- net BAT_8+: now also U$21.IN_VCC
Other:
- note added: "A DC-DC 12V"
- note added: "A DC-DC 24V"
- note added: "A Ordenador"
- note added: "Hacia el motor"
- note added: "I. General"
- note added: "Salida DC 5V"

Commit message: Actualización de esquema y pdf
Se crea un pdf para poder visualizar el esquema sin necesidad de Eagle
Parts:
- removed U$24: GPS, ecar:GPS
- added U$17: GPS, ecar:GPS
Connections:
- new net +48V->DC-DC12V: U$21.OUT+2, U$22.IN_+48V
- new net +48V->DC-DC24V: U$21.OUT+1, U$23.IN_+48V
- new net GND->DC-DC12V: U$21.OUT-2, U$22.IN_GND
- new net GND->DC-DC24V: U$21.OUT-1, U$23.IN_GND
- new net GND_DC-DC12V->FRONTAL: U$17.IN_GND, U$22.OUT_GND
- new net GND_DC-DC24V->FRONTAL: U$23.OUT2_GND
- new net GND_DC-DC24V->VOLTIMETROS: U$23.OUT1_GND, U$4.GND, U$5.GND, U$6.GND
- new net VCC_DC-DC12V->FRONTAL: U$17.IN_12V, U$22.OUT_+12V
- new net VCC_DC-DC24V->FRONTAL: U$23.OUT2_+24V
- new net VCC_DC-DC24V->VOLTIMETROS: U$23.OUT1_+24V, U$4.VCC, U$5.VCC, U$6.VCC
- net BAT_1: now also U$4.V-
- net BAT_8+: now also U$4.V+
Other:
- note added: "MALETERO ECARM"

Commit message: Actualización esquema y pdf
Se ha concluido el cableado actual del maletero del vehículo eCARM.
Parts:
- added D1: HLMP6, display-hp:HLMP6
Connections:
- net GND_DC-DC24V->VOLTIMETROS renamed GND_DC-DC24V->SENSORES
- net N$1 renamed BAT_5+
- net VCC_DC-DC24V->VOLTIMETROS renamed VCC_DC-DC24V->SENSORES
- new net AMARILLO_A2_M-: U$6.V-
- new net AMARILLO_AO+: U$2.AI6
- new net AMARILLO_U_VOLT3: U$2.AI7, U$6.VOUT
- new net AZUL_J1-22_LED+: D1.K
- new net AZUL_U_VOLT1: U$2.AI0, U$4.VOUT
- new net BLANCO_F2: U$5.V+
- new net MARRON_GND_VOLT2: U$2.AI10, U$5.VOUT_GND
- new net MARRON_J1-16_LED-: D1.A
- new net NARANJA_GND_U1: U$2.AI8, U$4.VOUT_GND
- new net NARANJA_VOUT_A2: U$2.AI13
- new net NEGRO_F1: U$5.V-
- new net ROJO_GND_VOLT3: U$2.AI15, U$6.VOUT_GND
- new net VERDE_A1_M+: U$6.V+
- new net VERDE_U_VOLT2: U$2.AI2, U$5.VOUT
- new net VERDE_VOUT_A1-M+: U$2.AI5
- net AMARILLO_OUTPUT_HONEYWELL: now also U$2.AI3
- net MARRON_VCC_HONEYWELL: now also U$2.+5V
- net NEGRO_-VCC_HONEYWELL: now also U$2.AI11, U$2.DGND1
- net ROJO_VOUT_LEM: now also U$2.AI1
- net VERDE_GND_LEM: now also U$2.AI9
Other:
- note added: "AZUL_VACIO(M2) MARRON_VACIO(M2)"
- note added: "BLANCO_24V"
- note added: "NEGRO"
- note added: "ROJO"

Commit message: Cableado Caja Blanca Finalizado
Parts:
- added U$24: ARDUINO_PRO, ecar:ARDUINO_PRO
- added U$36: LIBRE_DAQ, ecar:LIBRE_DAQ
- U$32: value ARDUINO_PRO -> RELE_ARDUINO; device ecar:ARDUINO_PRO -> ecar:RELE_ARDUINO
Connections:
- new net /CS_DAQ: U$24.9, U$36./CS
- new net 5V: U$24.VCC, U$33.5V
- new net AO+: U$36.AO0
- new net AO-: U$36.GND
- new net CS: U$24.A0, U$34.CS
- new net CTS: U$33.CTS
- new net DIR: U$24.4, U$34.DIR
- new net DTR: U$24.GRN, U$33.DTR
- new net ENC_ABS_CLK: U$24.A3
- new net ENC_ABS_CS: U$24.A1
- new net ENC_ABS_DO: U$24.A2
- new net ENC_INC_A: U$1.6.A, U$24.2
- new net ENC_INC_B: U$1.B, U$24.5
- new net ETHERNET_RBP: U$31.ETHERNET
- new net GND: U$1.3.GND, U$24.GND, U$24.GND1, U$32.GND, U$33.GND, U$34.GND1, U$36.GND0
- new net HDMI_RBP: U$31.HDMI
- new net IN1: U$24.8, U$32.IN1
- new net IN2: U$24.7, U$32.IN2
- new net K1C: U$32.K1C
- new net K1I: U$32.K1I
- new net K1O: U$32.K1O
- new net K2C: U$32.K2C
- new net K2I: U$32.K2I
- new net K2O: U$32.K2O
- new net MOSI_DAQ: U$24.13, U$36.MOSI
- new net MOTOR_DIRECCION_+: U$1.MOTOR+, U$34.OUT_A
- new net MOTOR_DIRECCION_-: U$1.MOTOR-, U$34.OUT_B
- new net N$1: U$31.USB1, U$33.USB
- new net N$3: U$34.5VOUT, U$34.VCS
- new net N.C.: U$1.1.NC, U$1.10.I, U$1.4.NC, U$1.5./A, U$1.7./B, U$1.9/I
- new net PWMH: U$24.6, U$34.PWMH
- new net RXD: U$24.TXO, U$33.RXD
- new net SCK_DAQ: U$24.11, U$36.SCK
- new net TXD: U$24.RXI, U$33.TXD
- new net VCC_5V: U$1.2.VCC, U$24.VCC0, U$32.VCC, U$36.5V
- new net VGA_PC: U$16.VGA, U$28.VGA
- net 5V_GND: now also U$31.GND
- net 5V_VCC: now also U$31.VCC
- net GND_DC-DC12V->FRONTAL: now also U$34.GND-
- net VCC_DC-DC12V->FRONTAL: now also U$34.VCC+
Other:
- note added: "Manguera_Encoder_Absoluto"
- note added: "Manguera_Encoder_Incremental"
- moved on the sheet: U$7
