File: esquemas/Esquema_general.sch (EAGLE design)
At the start: 37 parts

Commit message: Cableado completo Caja Blanca
Parts:
- removed U$33: CONVERSOR_ARDUINO, ecar:CONVERSOR_ARDUINO
- U$24: value ARDUINO_PRO -> CLARAQUINO_V1.0; device ecar:ARDUINO_PRO -> ecar:CLARAQUINO_V1.0
Connections:
- removed net 5V: U$24.VCC, U$33.5V
- removed net CTS: U$33.CTS
- removed net DTR: U$24.GRN, U$33.DTR
- removed net IN2: U$24.7, U$32.IN2
- removed net N$1: U$31.USB1, U$33.USB
- removed net RXD: U$24.TXO, U$33.RXD
- removed net TXD: U$24.RXI, U$33.TXD
- new net USB: U$24.USB, U$31.USB1
- net /CS_DAQ: now also U$24.B4; no longer U$24.9
- net DIR: now also U$24.D6; no longer U$24.4
- net ENC_ABS_CLK: now also U$24.B1; no longer U$24.A3
- net ENC_ABS_CS: now also U$24.B0; no longer U$24.A1
- net ENC_ABS_DO: now also U$24.B2; no longer U$24.A2
- net ENC_INC_A: now also U$24.RXD1; no longer U$24.2
- net ENC_INC_B: now also U$24.TXD1; no longer U$24.5
- net GND: now also U$24.PWR1; no longer U$24.GND, U$24.GND1, U$33.GND
- net IN1: now also U$24.A1; no longer U$24.8
- net MOSI_DAQ: now also U$24.B5; no longer U$24.13
- net PWMH: now also U$24.D7; no longer U$24.6
- net SCK_DAQ: now also U$24.B7; no longer U$24.11
- net VCC_5V: now also U$24.PWR0; no longer U$24.VCC0
Other:
- note added: "CAJA AZUL"
- note added: "CAJA BLANCA"

Commit message: Cableado actual del vehículo eCARM
Connections:
- net GND_DC-DC24V->FRONTAL: now also U$29.GND
- net VCC_DC-DC24V->FRONTAL: now also U$29.VCC
Other:
- moved on the sheet: U$7
